Commit message: ajout pelle

File: gillou/src/description/gillou.urdf (robot description, URDF)
Before this commit: robot gillou_bot, 7 links, 6 joints
Links:
- added link left_arm_link; collision box size=${arm_length} ${arm_width} ${arm_height}; visual box size=${arm_length} ${arm_width} ${arm_height}
- added link right_arm_link; collision box size=${arm_length} ${arm_width} ${arm_height}; visual box size=${arm_length} ${arm_width} ${arm_height}
Joints:
- added joint left_arm_joint: type fixed, parent base_link, child left_arm_link, origin xyz=0.30 0.20 -0.06 rpy=0 0 0.5
- added joint right_arm_joint: type fixed, parent base_link, child right_arm_link, origin xyz=0.30 -0.20 -0.06 rpy=0 0 -0.5

Commit message: pelle

File: gillou/src/description/gillou.urdf (robot description, URDF)
Before this commit: robot gillou_bot, 9 links, 8 joints
Links:
- removed link lidar_link
- added link door_link; collision box size=${door_length} ${door_width} ${door_height}; visual box size=${door_length} ${door_width} ${door_height}
- added link first_hook_link; collision cylinder length=${hook_width} radius=${hook_radius}; visual cylinder length=${hook_width} radius=${hook_radius}
- added link second_hook_link; collision cylinder length=${hook_width} radius=${hook_radius}; visual cylinder length=${hook2_width} radius=${hook_radius}
Joints:
- removed joint lidar_joint
- added joint door_joint: type fixed, parent second_hook_link, child door_link, origin xyz=0 0 -0.15 rpy=0 0.5 0
- added joint first_hook_joint: type fixed, parent base_link, child first_hook_link, origin xyz=0.18 0 0.16 rpy=0 1.2 0
- added joint second_hook_joint: type fixed, parent first_hook_link, child second_hook_link, origin xyz=0.15 0 0.20 rpy=0 -1.8 0

Commit message: ajout 2 roues folles sur gazebo

File: gillou/src/description/gillou.urdf (robot description, URDF)
Before this commit: robot gillou_bot, 12 links, 11 joints
Links:
- removed link front_caster
- added link front_caster_l; collision sphere radius=${(wheel_radius+wheel_zoff-(base_height/2))}; visual sphere radius=${(wheel_radius+wheel_zoff-(base_height/2))}
- added link front_caster_r; collision sphere radius=${(wheel_radius+wheel_zoff-(base_height/2))}; visual sphere radius=${(wheel_radius+wheel_zoff-(base_height/2))}
Joints:
- removed joint caster_joint
- added joint caster_joint_l: type fixed, parent base_link, child front_caster_l, origin xyz=${caster_xoff} ${(0.5*base_width)/2} ${-(base_height/2)} rpy=0 0 0
- added joint caster_joint_r: type fixed, parent base_link, child front_caster_r, origin xyz=${caster_xoff} ${-(0.5*base_width)/2} ${-(base_height/2)} rpy=0 0 0

Commit message: maj pelle

File: gillou/src/description/gillou.urdf (robot description, URDF)
Before this commit: robot gillou_bot, 12 links, 11 joints
Joints:
- joint rot_joint_joint: axis (none) -> 0 0 1; limit (none) -> lower=-3.14 upper=3.14 effort=100 velocity=30; type fixed -> revolute

Commit message: robot marche arriere et avant propre

File: gillou/src/description/gillou.urdf (robot description, URDF)
Before this commit: robot gillou_bot, 13 links, 12 joints
Joints:
- joint caster_joint_l: type fixed -> continuous
- joint caster_joint_r: type fixed -> continuous
- joint rot_joint_joint: origin xyz=0.02 0 0.11 rpy=${pi/2} 0 0 -> xyz=0.02 0 0.11 rpy=${pi/2} -0.5 0

Commit message: push all

File: gillou/src/description/gillou.urdf (robot description, URDF)
Before this commit: robot gillou_bot, 13 links, 12 joints
Links:
- link base_link: geometry collision box size=${base_length} ${base_width} ${base_height}; visual mesh filename=package://gillou/description_inventor/robot.dae
- link first_hook_link: geometry collision cylinder length=${hook_width} radius=${hook_radius}; visual mesh filename=package://gillou/description_inventor/pelle.dae

Commit message: mesh mal placés

File: gillou/src/description/gillou.urdf (robot description, URDF)
Before this commit: robot gillou_bot, 13 links, 12 joints
Links:
- link base_link: geometry collision box size=${base_length} ${base_width} ${base_height}; visual mesh filename=file://$(find gillou)/src/description/description_inventor/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 scale=0.01 0.01 0.01
- link door_link: geometry collision box size=${door_length} ${door_width} ${door_height}
- link rot_joint_link: geometry collision cylinder length=${rot_joint_width} radius=${rot_joint_radius}; visual mesh filename=file://$(find gillou)/src/description/description_inventor/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 scale=0.01 0.01 0.01

Commit message: mesh ok

File: gillou/src/description/gillou.urdf (robot description, URDF)
Before this commit: robot gillou_bot, 13 links, 12 joints
Links:
- link door_link: geometry collision box size=${door_length} ${door_width} ${door_height}; visual box size=${door_length} ${door_width} ${door_height}
Joints:
- joint rot_joint_joint: origin xyz=0.02 0 0.11 rpy=${pi/2} -0.5 0 -> xyz=0.06 0 0.11 rpy=${pi/2} -0.5 0

Commit message: pelle-roue

File: gillou/src/description/gillou.urdf (robot description, URDF)
Before this commit: robot gillou_bot, 13 links, 12 joints
Links:
- link base_link: geometry collision box size=${base_length} ${base_width} ${base_height}; visual box size=${base_length} ${base_width} ${base_height}
- link door_link: geometry collision box size=${door_length} ${door_width} ${door_height}; visual box size=${door_length} ${door_width} ${door_height}
- link rot_joint_link: geometry collision cylinder length=${rot_joint_width} radius=${rot_joint_radius}; visual cylinder length=${rot_joint_width} radius=${rot_joint_radius}
Joints:
- joint rot_joint_joint: axis 0 0 1 -> (none); limit lower=-3.14 upper=3.14 effort=100 velocity=30 -> (none); origin xyz=0.02 0 0.11 rpy=${pi/2} -0.5 0 -> xyz=0 0 0 rpy=${pi/2} -0.5 0; parent base_link -> pelle_l_link; type revolute -> fixed

Commit message: tracking ne termine pas

File: gillou/src/description/gillou.urdf (robot description, URDF)
Before this commit: robot gillou_bot, 13 links, 12 joints
Links:
- link first_hook_link: geometry collision cylinder length=${hook_width} radius=${hook_radius}
- link rot_joint_link: geometry collision cylinder length=${rot_joint_width} radius=${rot_joint_radius}

Commit message: maj po

File: gillou/src/description/gillou.urdf (robot description, URDF)
Before this commit: robot gillou_bot, 13 links, 12 joints
Links:
- link first_hook_link: geometry collision cylinder length=${hook_width} radius=${hook_radius}; visual cylinder length=${hook_width} radius=${hook_radius}
- link rot_joint_link: geometry collision cylinder length=${rot_joint_width} radius=${rot_joint_radius}
